File: KiCad Files/simply_wearable/simply_wearable.kicad_sch (KiCad schematic)
At the start: 16 parts, among them J1 Conn_01x02_Socket, J2 1027 Motor, J3 Conn_01x07_Socket, J4 Conn_01x05_Socket, Q1 AO3400A, SW1 SW_Push, SW2 SW_Push, U1 nice_nano, U2 ER_OLEDM0.91_1x-I2C

Commit message: Day 2 Work (journal)
Parts:
- removed C1: C_Small, Capacitor_SMD:C_0805_2012Metric_Pad1.18x1.45mm_HandSolder, symbol Device:C_Small
- removed D1: 1N4148W, Diode_SMD:D_SOD-123, symbol Diode:1N4148W
- removed J2: 1027 Motor, Connector_JST:JST_PH_S2B-PH-K_1x02_P2.00mm_Horizontal, symbol Connector:Conn_01x02_Socket
- removed Q1: AO3400A, Package_TO_SOT_SMD:SOT-23, symbol Transistor_FET:AO3400A
- removed R1: 220, Resistor_THT:R_Axial_DIN0207_L6.3mm_D2.5mm_P7.62mm_Horizontal, symbol Device:R
- removed R2: 10K, Resistor_THT:R_Axial_DIN0207_L6.3mm_D2.5mm_P7.62mm_Horizontal, symbol Device:R
- added C1: C, Capacitor_SMD:C_0805_2012Metric_Pad1.18x1.45mm_HandSolder, symbol Device:C
Connections:
- net BAT+: now also J1.1 (Pin_1); no longer J1.2 (Pin_2)
- net VCC: now also C1.1
- net GND: now reaches J3.3 (Pin_3), J3.7 (Pin_7), R4.2, SW1.2, SW2.2, U1.14 (GND), U2.1 (GND)
- net GND: now also J1.2 (Pin_2), C1.2; no longer J1.1 (Pin_1)
- net M=: no longer names the net of U1.10 (P0.11)
- no-connect marks 26 -> 27
Other:
- moved on the sheet: J1

Commit message: PCB Completed and Production Files Added
Connections:
- net VCC: now also U1.29 (BAT+)
- no-connect marks 27 -> 26
Changed lines of the file:
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@@
+	)
+	(junction
+		(at 142.24 72.39)
+		(diameter 0)
+		(color 0 0 0 0)
 	)
 	(junction
@@
 	)
 	(no_connect
-		(at 142.24 69.85)
-	)
-	(no_connect
 		(at 104.14 77.47)
 	)
@@
 		(pts
 			(xy 97.79 72.39) (xy 104.14 72.39)
+		)
+		(stroke
+			(width 0)
+			(type default)
+		)
+	)
+	(wire
+		(pts
+			(xy 142.24 69.85) (xy 142.24 72.39)
 		)
 		(stroke
@@
 		)
 		(instances
-			(project "Untitled"
+			(project "simply_wearable"
 				(path "/3262e707-f2b1-490b-9ca0-ca8904fc963b"
 					(reference "R4")
@@
 		)
 		(instances
-			(project "Untitled"
+			(project "simply_wearable"
 				(path "/3262e707-f2b1-490b-9ca0-ca8904fc963b"
 					(reference "C1")
@@
 		)
 		(instances
-			(project "Untitled"
+			(project "simply_wearable"
 				(path "/3262e707-f2b1-490b-9ca0-ca8904fc963b"
 					(reference "SW2")
@@
 		)
 		(instances
-			(project "Untitled"
+			(project "simply_wearable"
 				(path "/3262e707-f2b1-490b-9ca0-ca8904fc963b"
 					(reference "J3")
@@
 		)
 		(instances
-			(project "Untitled"
+			(project "simply_wearable"
 				(path "/3262e707-f2b1-490b-9ca0-ca8904fc963b"
 					(reference "R3")
@@
 		)
 		(instances
-			(project "Untitled"
+			(project "simply_wearable"
 				(path "/3262e707-f2b1-490b-9ca0-ca8904fc963b"
 					(reference "U2")
@@
 		)
 		(instances
-			(project "Untitled"
+			(project "simply_wearable"
 				(path "/3262e707-f2b1-490b-9ca0-ca8904fc963b"
 					(reference "S1")
@@
 		)
 		(instances
-			(project "Untitled"
+			(project "simply_wearable"
 				(path "/3262e707-f2b1-490b-9ca0-ca8904fc963b"
 					(reference "J4")
@@
 		)
 		(instances
-			(project "Untitled"
+			(project "simply_wearable"
 				(path "/3262e707-f2b1-490b-9ca0-ca8904fc963b"
 					(reference "U1")
@@
 		)
 		(instances
-			(project "Untitled"
+			(project "simply_wearable"
 				(path "/3262e707-f2b1-490b-9ca0-ca8904fc963b"
 					(reference "J1")
@@
 		)
 		(instances
-			(project "Untitled"
+			(project "simply_wearable"
 				(path "/3262e707-f2b1-490b-9ca0-ca8904fc963b"
 					(reference "SW1")
